Commit message: versão 4 rodas separadas

File: src/robot_model_pkg/urdf/car.xacro (robot description, xacro)
@@ -24,4 +24,10 @@
     <color rgba="1 1 0 1" />
   </material>
+  <gazebo>
+    <plugin name="gazebo_ros_control" filename="libgazebo_ros_control.so">
+      <robotNamespace>/car</robotNamespace>
+      <robotSimType>gazebo_ros_control/DefaultRobotHWSim</robotSimType>
+    </plugin>
+  </gazebo>
   <!-- Base Link -->
   <link name="dummy"> </link>
@@ -90,74 +96,165 @@
       rpy="0 0 0" />
   </joint>
-  <!-- Wheel Macro -->
-  <xacro:macro name="wheel" params="prefix x y roll">
-    <link name="${prefix}_link">
-      <visual>
-        <geometry>
-          <cylinder radius="${wheel_radius}" length="${wheel_length}" />
-        </geometry>
-        <material name="yellow" />
-      </visual>
-      <collision>
-        <geometry>
-          <cylinder radius="${wheel_radius}" length="${wheel_length}" />
-        </geometry>
-      </collision>
-      <inertial>
-        <mass value="${wheel_mass}" />
-        <inertia
-          ixx="${(wheel_mass/12) * (3*wheel_radius**2 + wheel_length**2)}"
-          ixy="0"
-          ixz="0"
-          iyy="${(wheel_mass/12) * (3*wheel_radius**2 + wheel_length**2)}"
-          iyz="0"
-          izz="${(wheel_mass/2) * wheel_radius**2}" />
-      </inertial>
-    </link>
-    <joint name="${prefix}_joint" type="continuous">
-      <parent link="base_link" />
-      <child link="${prefix}_link" />
-      <origin xyz="${x} ${y} ${-car_height/2}" rpy="${roll} 0 0" />
-      <axis xyz="0 0 1" />
-      <limit effort="10.0" velocity="10.0" />
+  <!-- Wheels -->
+  <!-- front_left_wheel -->
+  <link name="front_left_wheel_link">
+    <visual>
+      <geometry>
+        <cylinder radius="${wheel_radius}" length="${wheel_length}" />
+      </geometry>
+      <material name="yellow" />
+    </visual>
+    <collision>
+      <geometry>
+        <cylinder radius="${wheel_radius}" length="${wheel_length}" />
+      </geometry>
+    </collision>
+    <inertial>
+      <mass value="${wheel_mass}" />
+      <inertia
+        ixx="${(wheel_mass/12) * (3*wheel_radius**2 + wheel_length**2)}"
+        ixy="0"
+        ixz="0"
+        iyy="${(wheel_mass/12) * (3*wheel_radius**2 + wheel_length**2)}"
+        iyz="0"
+        izz="${(wheel_mass/2) * wheel_radius**2}" />
+    </inertial>
+  </link>
+  <joint name="front_left_wheel_joint" type="continuous">
+    <parent link="base_link" />
+    <child link="front_left_wheel_link" />
+    <origin xyz="${car_length/2} ${car_width/2+wheel_length/2} ${-car_height/2}" rpy="${pi/2} 0 0" />
+    <axis xyz="0 0 1" />
+    <limit effort="10.0" velocity="10.0" />
+  </joint>
+  <!-- front_right_wheel -->
+  <link name="front_right_wheel_link">
+    <visual>
+      <geometry>
+        <cylinder radius="${wheel_radius}" length="${wheel_length}" />
+      </geometry>
+      <material name="yellow" />
+    </visual>
+    <collision>
+      <geometry>
+        <cylinder radius="${wheel_radius}" length="${wheel_length}" />
+      </geometry>
+    </collision>
+    <inertial>
+      <mass value="${wheel_mass}" />
+      <inertia
+        ixx="${(wheel_mass/12) * (3*wheel_radius**2 + wheel_length**2)}"
+        ixy="0"
+        ixz="0"
+        iyy="${(wheel_mass/12) * (3*wheel_radius**2 + wheel_length**2)}"
+        iyz="0"
+        izz="${(wheel_mass/2) * wheel_radius**2}" />
+    </inertial>
+  </link>
+  <joint name="front_right_wheel_joint" type="continuous">
+    <parent link="base_link" />
+    <child link="front_right_wheel_link" />
+    <origin xyz="${car_length/2} ${-car_width/2-wheel_length/2} ${-car_height/2}" rpy="${pi/2} 0 0" />
+    <axis xyz="0 0 1" />
+    <limit effort="10.0" velocity="10.0" />
+  </joint>
+  <!-- back_left_wheel -->
+  <link name="back_left_wheel_link">
+    <visual>
+      <geometry>
+        <cylinder radius="${wheel_radius}" length="${wheel_length}" />
+      </geometry>
+      <material name="yellow" />
+    </visual>
+    <collision>
+      <geometry>
+        <cylinder radius="${wheel_radius}" length="${wheel_length}" />
+      </geometry>
+    </collision>
+    <inertial>
+      <mass value="${wheel_mass}" />
+      <inertia
+        ixx="${(wheel_mass/12) * (3*wheel_radius**2 + wheel_length**2)}"
+        ixy="0"
+        ixz="0"
+        iyy="${(wheel_mass/12) * (3*wheel_radius**2 + wheel_length**2)}"
+        iyz="0"
+        izz="${(wheel_mass/2) * wheel_radius**2}" />
+    </inertial>
+  </link>
+  <joint name="back_left_wheel_joint" type="continuous">
+    <parent link="base_link" />
+    <child link="back_left_wheel_link" />
+    <origin xyz="${-car_length/2} ${+car_width/2+wheel_length/2} ${-car_height/2}" rpy="${pi/2} 0 0" />
+    <axis xyz="0 0 1" />
+    <limit effort="10.0" velocity="10.0" />
+  </joint>
+  <!-- back_right_wheel -->
+  <link name="back_right_wheel_link">
+    <visual>
+      <geometry>
+        <cylinder radius="${wheel_radius}" length="${wheel_length}" />
+      </geometry>
+      <material name="yellow" />
+    </visual>
+    <collision>
+      <geometry>
+        <cylinder radius="${wheel_radius}" length="${wheel_length}" />
+      </geometry>
+    </collision>
+    <inertial>
+      <mass value="${wheel_mass}" />
+      <inertia
+        ixx="${(wheel_mass/12) * (3*wheel_radius**2 + wheel_length**2)}"
+        ixy="0"
+        ixz="0"
+        iyy="${(wheel_mass/12) * (3*wheel_radius**2 + wheel_length**2)}"
+        iyz="0"
+        izz="${(wheel_mass/2) * wheel_radius**2}" />
+    </inertial>
+  </link>
+  <joint name="back_right_wheel_joint" type="continuous">
+    <parent link="base_link" />
+    <child link="back_right_wheel_link" />
+    <origin xyz="${-car_length/2} ${-car_width/2-wheel_length/2} ${-car_height/2}"
+      rpy="${pi/2} 0 0" />
+    <axis xyz="0 0 1" />
+    <limit effort="10.0" velocity="10.0" />
+  </joint>
+  <transmission name="back_left_wheel_trans">
+    <type>transmission_interface/SimpleTransmission</type>
+    <joint name="back_left_wheel_joint">
+      <hardwareInterface>hardware_interface/EffortJointInterface</hardwareInterface>
     </joint>
-    <gazebo reference="${prefix}_link">
-      <mu1>1.0</mu1>
-      <mu2>1.0</mu2>
-      <!-- <kp>1000000.0</kp>
-      <kd>1.0</kd> -->
-    </gazebo>
-  </xacro:macro>
-  <!-- 4 wheels -->
-  <xacro:wheel prefix="front_left_wheel" x="${car_length/2}" y="${car_width/2+wheel_length/2}"
-    roll="${pi/2}" />
-  <xacro:wheel prefix="front_right_wheel" x="${car_length/2}" y="${-car_width/2-wheel_length/2}"
-    roll="${pi/2}" />
-  <xacro:wheel prefix="back_left_wheel" x="${-car_length/2}" y="${+car_width/2+wheel_length/2}"
-    roll="${pi/2}" />
-  <xacro:wheel prefix="back_right_wheel" x="${-car_length/2}" y="${-car_width/2-wheel_length/2}"
-    roll="${pi/2}" />
-  <!-- Gazebo ROS Control -->
-  <!-- <gazebo>
-    <plugin name="gazebo_ros_control" filename="libgazebo_ros_control.so">
-      <controlPeriod>0.001</controlPeriod>
-      <robotSimType>gazebo_ros_control/DefaultRobotHWSim</robotSimType>
-    </plugin>
-  </gazebo> -->
-  <gazebo>
-    <plugin name="differential_drive_controller" filename="libgazebo_ros_diff_drive.so">
-      <updateRate>50.0</updateRate>
-      <leftJoint>front_left_wheel_joint</leftJoint>
-      <rightJoint>front_right_wheel_joint</rightJoint>
-      <wheelSeparation>0.2124</wheelSeparation>
-      <wheelDiameter>0.1016</wheelDiameter>
-      <robotBaseFrame>base_link</robotBaseFrame>
-      <odometryFrame>odom</odometryFrame>
-      <odometryTopic>odom</odometryTopic>
-      <commandTopic>cmd_vel</commandTopic>
-      <publishOdomTF>true</publishOdomTF>
-      <publishWheelJointState>true</publishWheelJointState>
-      <legacyMode>false</legacyMode>
-    </plugin>
+    <actuator name="back_left_wheel_motor">
+      <hardwareInterface>hardware_interface/EffortJointInterface</hardwareInterface>
+      <mechanicalReduction>1</mechanicalReduction>
+    </actuator>
+  </transmission>
+  <transmission name="back_right_wheel_trans">
+    <type>transmission_interface/SimpleTransmission</type>
+    <joint name="back_right_wheel_joint">
+      <hardwareInterface>hardware_interface/EffortJointInterface</hardwareInterface>
+    </joint>
+    <actuator name="back_right_wheel_motor">
+      <hardwareInterface>hardware_interface/EffortJointInterface</hardwareInterface>
+      <mechanicalReduction>1</mechanicalReduction>
+    </actuator>
+  </transmission>
+  <gazebo reference="back_right_wheel_link">
+    <mu1>1.0</mu1>
+    <mu2>1.0</mu2>
+  </gazebo>
+  <gazebo reference="back_left_wheel_link">
+    <mu1>1.0</mu1>
+    <mu2>1.0</mu2>
+  </gazebo>
+  <gazebo reference="front_right_wheel_link">
+    <mu1>1.0</mu1>
+    <mu2>1.0</mu2>
+  </gazebo>
+  <gazebo reference="front_left_wheel_link">
+    <mu1>1.0</mu1>
+    <mu2>1.0</mu2>
   </gazebo>
 </robot>

Commit message: Commands added and the steering joint configurated

File: src/robot_model_pkg/urdf/car.xacro (robot description, xacro)
@@ -97,66 +97,92 @@
   </joint>
   <!-- Wheels -->
-  <!-- front_left_wheel -->
-  <link name="front_left_wheel_link">
-    <visual>
-      <geometry>
-        <cylinder radius="${wheel_radius}" length="${wheel_length}" />
-      </geometry>
-      <material name="yellow" />
-    </visual>
-    <collision>
-      <geometry>
-        <cylinder radius="${wheel_radius}" length="${wheel_length}" />
-      </geometry>
-    </collision>
-    <inertial>
-      <mass value="${wheel_mass}" />
-      <inertia
-        ixx="${(wheel_mass/12) * (3*wheel_radius**2 + wheel_length**2)}"
-        ixy="0"
-        ixz="0"
-        iyy="${(wheel_mass/12) * (3*wheel_radius**2 + wheel_length**2)}"
-        iyz="0"
-        izz="${(wheel_mass/2) * wheel_radius**2}" />
-    </inertial>
-  </link>
-  <joint name="front_left_wheel_joint" type="continuous">
-    <parent link="base_link" />
-    <child link="front_left_wheel_link" />
-    <origin xyz="${car_length/2} ${car_width/2+wheel_length/2} ${-car_height/2}" rpy="${pi/2} 0 0" />
-    <axis xyz="0 0 1" />
-    <limit effort="10.0" velocity="10.0" />
-  </joint>
-  <!-- front_right_wheel -->
-  <link name="front_right_wheel_link">
-    <visual>
-      <geometry>
-        <cylinder radius="${wheel_radius}" length="${wheel_length}" />
-      </geometry>
-      <material name="yellow" />
-    </visual>
-    <collision>
-      <geometry>
-        <cylinder radius="${wheel_radius}" length="${wheel_length}" />
-      </geometry>
-    </collision>
-    <inertial>
-      <mass value="${wheel_mass}" />
-      <inertia
-        ixx="${(wheel_mass/12) * (3*wheel_radius**2 + wheel_length**2)}"
-        ixy="0"
-        ixz="0"
-        iyy="${(wheel_mass/12) * (3*wheel_radius**2 + wheel_length**2)}"
-        iyz="0"
-        izz="${(wheel_mass/2) * wheel_radius**2}" />
-    </inertial>
-  </link>
-  <joint name="front_right_wheel_joint" type="continuous">
-    <parent link="base_link" />
-    <child link="front_right_wheel_link" />
-    <origin xyz="${car_length/2} ${-car_width/2-wheel_length/2} ${-car_height/2}" rpy="${pi/2} 0 0" />
-    <axis xyz="0 0 1" />
-    <limit effort="10.0" velocity="10.0" />
-  </joint>
+  <!-- Front Left Wheel -->
+<link name="front_left_steer_link">
+  <inertial>
+    <mass value="0.1"/>
+    <inertia ixx="0.001" ixy="0.0" ixz="0.0" iyy="0.001" iyz="0.0" izz="0.001"/>
+  </inertial>
+</link>
+<link name="front_left_wheel_link">
+  <visual>
+    <geometry>
+      <cylinder radius="${wheel_radius}" length="${wheel_length}"/>
+    </geometry>
+    <material name="yellow"/>
+  </visual>
+  <collision>
+    <geometry>
+      <cylinder radius="${wheel_radius}" length="${wheel_length}"/>
+    </geometry>
+  </collision>
+  <inertial>
+    <mass value="${wheel_mass}"/>
+    <inertia
+      ixx="${(wheel_mass/12) * (3*wheel_radius**2 + wheel_length**2)}"
+      ixy="0" ixz="0"
+      iyy="${(wheel_mass/12) * (3*wheel_radius**2 + wheel_length**2)}"
+      iyz="0"
+      izz="${(wheel_mass/2) * wheel_radius**2}"/>
+  </inertial>
+</link>
+<!-- Steering joint (connects base to steer link) -->
+<joint name="steer_front_left_joint" type="revolute">
+  <parent link="base_link"/>
+  <child link="front_left_steer_link"/>
+  <origin xyz="${car_length/2} ${car_width/2} ${-car_height/2}"/>
+  <axis xyz="0 0 1"/>
+  <limit lower="-0.785" upper="0.785" effort="10.0" velocity="10.0"/> <!-- ±45° -->
+</joint>
+<!-- Wheel joint (connects steer link to wheel, provides rotation) -->
+<joint name="front_left_wheel_joint" type="continuous">
+  <parent link="front_left_steer_link"/>
+  <child link="front_left_wheel_link"/>
+  <origin xyz="0 ${wheel_length/2} 0" rpy="${pi/2} 0 0"/>
+  <axis xyz="0 0 1"/>
+</joint>
+<!-- Front Right Wheel -->
+<link name="front_right_steer_link">
+  <inertial>
+    <mass value="0.1"/>
+    <inertia ixx="0.001" ixy="0.0" ixz="0.0" iyy="0.001" iyz="0.0" izz="0.001"/>
+  </inertial>
+</link>
+<link name="front_right_wheel_link">
+  <visual>
+    <geometry>
+      <cylinder radius="${wheel_radius}" length="${wheel_length}"/>
+    </geometry>
+    <material name="yellow"/>
+  </visual>
+  <collision>
+    <geometry>
+      <cylinder radius="${wheel_radius}" length="${wheel_length}"/>
+    </geometry>
+  </collision>
+  <inertial>
+    <mass value="${wheel_mass}"/>
+    <inertia
+      ixx="${(wheel_mass/12) * (3*wheel_radius**2 + wheel_length**2)}"
+      ixy="0" ixz="0"
+      iyy="${(wheel_mass/12) * (3*wheel_radius**2 + wheel_length**2)}"
+      iyz="0"
+      izz="${(wheel_mass/2) * wheel_radius**2}"/>
+  </inertial>
+</link>
+<!-- Steering joint (connects base to steer link) -->
+<joint name="steer_front_right_joint" type="revolute">
+  <parent link="base_link"/>
+  <child link="front_right_steer_link"/>
+  <origin xyz="${car_length/2} ${-car_width/2} ${-car_height/2}"/>
+  <axis xyz="0 0 1"/>
+  <limit lower="-0.785" upper="0.785" effort="10.0" velocity="10.0"/> <!-- ±45° -->
+</joint>
+<!-- Wheel joint (connects steer link to wheel, provides rotation) -->
+<joint name="front_right_wheel_joint" type="continuous">
+  <parent link="front_right_steer_link"/>
+  <child link="front_right_wheel_link"/>
+  <origin xyz="0 ${-wheel_length/2} 0" rpy="${pi/2} 0 0"/>
+  <axis xyz="0 0 1"/>
+</joint>
   <!-- back_left_wheel -->
   <link name="back_left_wheel_link">

Commit message: The car can turn, but the steering wheels are still independent

File: src/robot_model_pkg/urdf/car.xacro (robot description, xacro)
@@ -268,19 +268,39 @@
     </actuator>
   </transmission>
+  <transmission name="front_left_steer_trans">
+    <type>transmission_interface/SimpleTransmission</type>
+    <joint name="steer_front_left_joint">
+      <hardwareInterface>hardware_interface/EffortJointInterface</hardwareInterface>
+    </joint>
+    <actuator name="front_left_steer_motor">
+      <hardwareInterface>hardware_interface/EffortJointInterface</hardwareInterface>
+      <mechanicalReduction>1</mechanicalReduction>
+    </actuator>
+  </transmission>
+  <transmission name="front_right_steer_trans">
+    <type>transmission_interface/SimpleTransmission</type>
+    <joint name="steer_front_right_joint">
+      <hardwareInterface>hardware_interface/EffortJointInterface</hardwareInterface>
+    </joint>
+    <actuator name="front_right_steer_motor">
+      <hardwareInterface>hardware_interface/EffortJointInterface</hardwareInterface>
+      <mechanicalReduction>1</mechanicalReduction>
+    </actuator>
+  </transmission>
   <gazebo reference="back_right_wheel_link">
-    <mu1>1.0</mu1>
-    <mu2>1.0</mu2>
+    <mu1>5.0</mu1>
+    <mu2>5.0</mu2>
   </gazebo>
   <gazebo reference="back_left_wheel_link">
-    <mu1>1.0</mu1>
-    <mu2>1.0</mu2>
+    <mu1>5.0</mu1>
+    <mu2>5.0</mu2>
   </gazebo>
   <gazebo reference="front_right_wheel_link">
-    <mu1>1.0</mu1>
-    <mu2>1.0</mu2>
+    <mu1>5.0</mu1>
+    <mu2>5.0</mu2>
   </gazebo>
   <gazebo reference="front_left_wheel_link">
-    <mu1>1.0</mu1>
-    <mu2>1.0</mu2>
+    <mu1>5.0</mu1>
+    <mu2>5.0</mu2>
   </gazebo>
 </robot>
