Commit message: control is perfect

File: src/steering_car/urdf/car.xacro (robot description, xacro)
@@ -14,6 +14,9 @@
   <xacro:property name="capota_car_mass" value="0.3" />
   <xacro:property name="steering_cylinder_radius" value="0.01" />
-  <xacro:property name="steering_cylinder_length" value="0.25" />
+  <xacro:property name="steering_cylinder_length" value="0.2124" />
   <xacro:property name="steering_cylinder_mass" value="0.05" />
+<!-- control parameters -->
+  <xacro:property name="back_wheels_velocity_limit" value="100.0" />
+  <xacro:property name="steering_velocity_limit" value="5.0" />
   <material name="green">
     <color rgba="0 1 0 1" />
@@ -34,5 +37,5 @@
     </plugin>
   </gazebo>
-  <!-- Base Link -->
+  <!-- Dummy and Base Link -->
   <link name="dummy"> </link>
   <joint name="dummy_joint" type="fixed">
@@ -63,9 +66,5 @@
     </inertial>
   </link>
-  <!-- Gazebo friction parameters -->
-  <gazebo reference="base_link">
-    <mu1>0.2</mu1>
-    <mu2>0.2</mu2>
-  </gazebo>
+<!-- Capota of car -->
   <link name="capota">
     <visual>
@@ -97,29 +96,36 @@
       rpy="0 0 0" />
   </joint>
+<!-- Steering cylinder axis -->
+<link name="steering_cylinder_link">
+    <visual>
+      <geometry>
+        <cylinder radius="${steering_cylinder_radius}" length="${steering_cylinder_length}"/>
+      </geometry>
+      <material name="grey"/>
+    </visual>
+    <collision>
+      <geometry>
+        <cylinder radius="${steering_cylinder_radius}" length="${steering_cylinder_length}"/>
+      </geometry>
+    </collision>
+    <inertial>
+      <mass value="${steering_cylinder_mass}"/>
+      <inertia
+        ixx="${(steering_cylinder_mass/12) * (3*steering_cylinder_radius**2 + steering_cylinder_length**2)}"
+        ixy="0" ixz="0"
+        iyy="${(steering_cylinder_mass/12) * (3*steering_cylinder_radius**2 + steering_cylinder_length**2)}"
+        iyz="0"
+        izz="${(steering_cylinder_mass/2) * steering_cylinder_radius**2}"/>
+    </inertial>
+  </link>
+  <joint name="steering_cylinder_joint" type="revolute">
+    <parent link="base_link"/>
+    <child link="steering_cylinder_link"/>
+    <origin xyz="${car_length/2-car_length/16} 0  ${-car_height/2}" rpy="${pi/2} 0 0"/>
+    <axis xyz="0 1 0"/>
+    <limit lower="${-pi/16}" upper="${pi/16}" effort="10.0" velocity="${steering_velocity_limit}"/>
+  </joint>
   <!-- Wheels -->
   <!-- Front Left Wheel -->
- <link name="front_steer_assembly_link">
-    <inertial>
-      <mass value="0.2"/>
-      <inertia ixx="0.002" ixy="0.0" ixz="0.0" iyy="0.002" iyz="0.0" izz="0.002"/>
-    </inertial>
-  </link>
-  <joint name="front_steer_joint" type="revolute">
-    <parent link="base_link"/>
-    <child link="front_steer_assembly_link"/>
-    <origin xyz="${car_length/2} 0 ${-car_height/2}"/>
-    <axis xyz="0 0 1"/>
-    <limit lower="-0.785" upper="0.785" effort="20.0" velocity="10.0"/> </joint>
-  <link name="front_left_steer_link">
-    <inertial>
-      <mass value="0.1"/>
-      <inertia ixx="0.001" ixy="0.0" ixz="0.0" iyy="0.001" iyz="0.0" izz="0.001"/>
-    </inertial>
-  </link>
-  <joint name="front_left_steer_fixed_joint" type="fixed">
-    <parent link="front_steer_assembly_link"/>
-    <child link="front_left_steer_link"/>
-    <origin xyz="0 ${car_width/2} 0"/>
-  </joint>
   <link name="front_left_wheel_link">
     <visual>
@@ -145,21 +151,10 @@
   </link>
   <joint name="front_left_wheel_joint" type="continuous">
-    <parent link="front_left_steer_link"/>
+    <parent link="steering_cylinder_link"/>
     <child link="front_left_wheel_link"/>
-    <origin xyz="0 ${wheel_length/2} 0" rpy="${pi/2} 0 0"/>
+    <origin xyz="0 0 ${steering_cylinder_length/2+wheel_length/2}" rpy="0 0 0"/>
     <axis xyz="0 0 1"/>
   </joint>
 <!-- Front Right Wheel -->
-  <link name="front_right_steer_link">
-    <inertial>
-      <mass value="0.1"/>
-      <inertia ixx="0.001" ixy="0.0" ixz="0.0" iyy="0.001" iyz="0.0" izz="0.001"/>
-    </inertial>
-  </link>
-  <joint name="front_right_steer_fixed_joint" type="fixed">
-    <parent link="front_steer_assembly_link"/>
-    <child link="front_right_steer_link"/>
-    <origin xyz="0 ${-car_width/2} 0"/>
-  </joint>
   <link name="front_right_wheel_link">
     <visual>
@@ -185,35 +180,8 @@
   </link>
   <joint name="front_right_wheel_joint" type="continuous">
-    <parent link="front_right_steer_link"/>
+    <parent link="steering_cylinder_link"/>
     <child link="front_right_wheel_link"/>
-    <origin xyz="0 ${-wheel_length/2} 0" rpy="${pi/2} 0 0"/>
+    <origin xyz="0 0 ${-steering_cylinder_length/2-wheel_length/2} " rpy="0 0 0"/>
     <axis xyz="0 0 1"/>
-  </joint>
-<link name="steering_cylinder_link">
-    <visual>
-      <geometry>
-        <cylinder radius="${steering_cylinder_radius}" length="${steering_cylinder_length}"/>
-      </geometry>
-      <material name="grey"/>
-    </visual>
-    <collision>
-      <geometry>
-        <cylinder radius="${steering_cylinder_radius}" length="${steering_cylinder_length}"/>
-      </geometry>
-    </collision>
-    <inertial>
-      <mass value="${steering_cylinder_mass}"/>
-      <inertia
-        ixx="${(steering_cylinder_mass/12) * (3*steering_cylinder_radius**2 + steering_cylinder_length**2)}"
-        ixy="0" ixz="0"
-        iyy="${(steering_cylinder_mass/12) * (3*steering_cylinder_radius**2 + steering_cylinder_length**2)}"
-        iyz="0"
-        izz="${(steering_cylinder_mass/2) * steering_cylinder_radius**2}"/>
-    </inertial>
-  </link>
-  <joint name="steering_cylinder_joint" type="fixed">
-    <parent link="front_right_steer_link"/>
-    <child link="steering_cylinder_link"/>
-    <origin xyz="0 ${steering_cylinder_length/2} 0" rpy="${pi/2} 0 0"/>
   </joint>
   <!-- back_left_wheel -->
@@ -246,5 +214,5 @@
     <origin xyz="${-car_length/2} ${+car_width/2+wheel_length/2} ${-car_height/2}" rpy="${pi/2} 0 0" />
     <axis xyz="0 0 1" />
-    <limit effort="10.0" velocity="10.0" />
+    <limit effort="10.0" velocity="${back_wheels_velocity_limit}" />
   </joint>
   <!-- back_right_wheel -->
@@ -278,5 +246,5 @@
       rpy="${pi/2} 0 0" />
     <axis xyz="0 0 1" />
-    <limit effort="10.0" velocity="10.0" />
+    <limit effort="10.0" velocity="${back_wheels_velocity_limit}" />
   </joint>
   <transmission name="back_left_wheel_trans">
@@ -302,5 +270,5 @@
   <transmission name="front_steer_trans">
     <type>transmission_interface/SimpleTransmission</type>
-    <joint name="front_steer_joint">
+    <joint name="steering_cylinder_joint">
       <hardwareInterface>hardware_interface/EffortJointInterface</hardwareInterface>
     </joint>
@@ -310,4 +278,9 @@
     </actuator>
   </transmission>
+  <!-- Gazebo friction parameters -->
+  <gazebo reference="base_link">
+    <mu1>0.2</mu1>
+    <mu2>0.2</mu2>
+  </gazebo>
   <gazebo reference="back_right_wheel_link">
     <mu1>5.0</mu1>

Commit message: car camera insert

File: src/steering_car/urdf/car.xacro (robot description, xacro)
@@ -248,4 +248,59 @@
     <limit effort="10.0" velocity="${back_wheels_velocity_limit}" />
   </joint>
+<!-- Camera -->
+<link name="camera_link">
+    <visual>
+      <geometry>
+        <box size="0.02 0.02 0.02"/> </geometry>
+      <material name="grey"/>
+    </visual>
+    <collision>
+      <geometry>
+        <box size="0.02 0.02 0.02"/>
+      </geometry>
+    </collision>
+    <inertial>
+      <mass value="0.01"/> <inertia ixx="0.00000833" ixy="0" ixz="0"
+               iyy="0.00000833" iyz="0"
+               izz="0.00000833"/>
+    </inertial>
+  </link>
+  <joint name="camera_joint" type="fixed">
+    <parent link="capota"/>
+    <child link="camera_link"/>
+    <origin xyz="${capota_car_width/2} 0 ${capota_car_height/2 + 0.002}" rpy="0 0 0"/>
+  </joint>
+<gazebo reference="camera_link">
+    <sensor type="camera" name="car_camera_sensor">
+      <update_rate>30.0</update_rate> <camera name="car_camera">
+        <horizontal_fov>1.39626</horizontal_fov> <image>
+          <width>640</width>
+          <height>480</height>
+          <format>R8G8B8</format>
+        </image>
+        <clip>
+          <near>0.05</near>
+          <far>10.0</far>
+        </clip>
+        <noise>
+          <type>gaussian</type>
+          <mean>0.0</mean>
+          <stddev>0.007</stddev>
+        </noise>
+      </camera>
+      <plugin name="camera_controller" filename="libgazebo_ros_camera.so">
+        <robotNamespace>/car</robotNamespace> <alwaysOn>true</alwaysOn>
+        <updateRate>30.0</updateRate>
+        <cameraName>car_camera</cameraName>
+        <imageTopicName>image_raw</imageTopicName>
+        <cameraInfoTopicName>camera_info</cameraInfoTopicName>
+        <frameName>camera_link_optical</frameName> <hackBaseline>0.07</hackBaseline> <distortionK1>0.0</distortionK1>
+        <distortionK2>0.0</distortionK2>
+        <distortionK3>0.0</distortionK3>
+        <distortionT1>0.0</distortionT1>
+        <distortionT2>0.0</distortionT2>
+      </plugin>
+    </sensor>
+  </gazebo>
   <transmission name="back_left_wheel_trans">
     <type>transmission_interface/SimpleTransmission</type>

Commit message: versao mais atualizada

File: src/steering_car/urdf/car.xacro (robot description, xacro)
@@ -5,5 +5,5 @@
   <xacro:property name="car_width" value="0.2124" />
   <xacro:property name="car_height" value="0.0762" />
-  <xacro:property name="car_mass" value="0.7" />
+  <xacro:property name="car_mass" value="1.4" />
   <xacro:property name="wheel_radius" value="0.0508" />
   <xacro:property name="wheel_length" value="0.0508" />
@@ -17,5 +17,5 @@
   <xacro:property name="steering_cylinder_mass" value="0.05" />
 <!-- control parameters -->
-  <xacro:property name="back_wheels_velocity_limit" value="100.0" />
+  <xacro:property name="back_wheels_velocity_limit" value="10.0" />
   <xacro:property name="steering_velocity_limit" value="5.0" />
   <material name="green">
@@ -345,18 +345,18 @@
   </gazebo>
   <gazebo reference="back_right_wheel_link">
-    <mu1>25.0</mu1>
-    <mu2>25.0</mu2>
+    <mu1>100.0</mu1>
+    <mu2>100.0</mu2>
   </gazebo>
   <gazebo reference="back_left_wheel_link">
-    <mu1>25.0</mu1>
-    <mu2>25.0</mu2>
+    <mu1>100.0</mu1>
+    <mu2>100.0</mu2>
   </gazebo>
   <gazebo reference="front_right_wheel_link">
-    <mu1>25.0</mu1>
-    <mu2>25.0</mu2>
+    <mu1>100.0</mu1>
+    <mu2>100.0</mu2>
   </gazebo>
   <gazebo reference="front_left_wheel_link">
-    <mu1>25.0</mu1>
-    <mu2>25.0</mu2>
+    <mu1>100.0</mu1>
+    <mu2>100.0</mu2>
   </gazebo>
 </robot>

Commit message: empirical upgrades

File: src/steering_car/urdf/car.xacro (robot description, xacro)
@@ -5,18 +5,39 @@
   <xacro:property name="car_width" value="0.2124" />
   <xacro:property name="car_height" value="0.0762" />
-  <xacro:property name="car_mass" value="1.4" />
+  <xacro:property name="car_mass" value="2.0" />
   <xacro:property name="wheel_radius" value="0.0508" />
   <xacro:property name="wheel_length" value="0.0508" />
-  <xacro:property name="wheel_mass" value="0.1" />
+  <xacro:property name="wheel_mass" value="0.4" />
   <xacro:property name="capota_car_length" value="0.2746" />      <!-- x axis  -->
   <xacro:property name="capota_car_width" value="0.2124" />       <!-- y axis  -->
   <xacro:property name="capota_car_height" value="0.0508" />      <!-- z axis  -->
-  <xacro:property name="capota_car_mass" value="0.3" />
+  <xacro:property name="capota_car_mass" value="0.25" />
   <xacro:property name="steering_cylinder_radius" value="0.01" />
   <xacro:property name="steering_cylinder_length" value="0.2124" />
   <xacro:property name="steering_cylinder_mass" value="0.05" />
 <!-- control parameters -->
-  <xacro:property name="back_wheels_velocity_limit" value="10.0" />
-  <xacro:property name="steering_velocity_limit" value="5.0" />
+  <xacro:property name="back_wheels_velocity_limit" value="100.0" />
+  <xacro:property name="steering_velocity_limit" value="100.0" />
+  <!-- Gazebo friction parameters -->
+  <gazebo reference="base_link">
+    <mu1>0.2</mu1>
+    <mu2>0.2</mu2>
+  </gazebo>
+  <gazebo reference="back_right_wheel_link">
+    <mu1>100.0</mu1>
+    <mu2>100.0</mu2>
+  </gazebo>
+  <gazebo reference="back_left_wheel_link">
+    <mu1>100.0</mu1>
+    <mu2>100.0</mu2>
+  </gazebo>
+  <gazebo reference="front_right_wheel_link">
+    <mu1>100.0</mu1>
+    <mu2>100.0</mu2>
+  </gazebo>
+  <gazebo reference="front_left_wheel_link">
+    <mu1>100.0</mu1>
+    <mu2>100.0</mu2>
+  </gazebo>
   <material name="green">
     <color rgba="0 1 0 1" />
@@ -130,5 +151,5 @@
     <origin xyz="${car_length/2-car_length/16} 0  ${-car_height/2}" rpy="${pi/2} 0 0"/>
     <axis xyz="0 1 0"/>
-    <limit lower="${-pi/16}" upper="${pi/16}" effort="10.0" velocity="${steering_velocity_limit}"/>
+    <limit lower="${-pi/8}" upper="${pi/8}" effort="10.0" velocity="${steering_velocity_limit}"/>
   </joint>
   <!-- Wheels -->
@@ -339,24 +360,3 @@
     </actuator>
   </transmission>
-  <!-- Gazebo friction parameters -->
-  <gazebo reference="base_link">
-    <mu1>0.2</mu1>
-    <mu2>0.2</mu2>
-  </gazebo>
-  <gazebo reference="back_right_wheel_link">
-    <mu1>100.0</mu1>
-    <mu2>100.0</mu2>
-  </gazebo>
-  <gazebo reference="back_left_wheel_link">
-    <mu1>100.0</mu1>
-    <mu2>100.0</mu2>
-  </gazebo>
-  <gazebo reference="front_right_wheel_link">
-    <mu1>100.0</mu1>
-    <mu2>100.0</mu2>
-  </gazebo>
-  <gazebo reference="front_left_wheel_link">
-    <mu1>100.0</mu1>
-    <mu2>100.0</mu2>
-  </gazebo>
 </robot>

Commit message: version 2.3

File: src/steering_car/urdf/car.xacro (robot description, xacro)
@@ -9,15 +9,10 @@
   <xacro:property name="wheel_length" value="0.0508" />
   <xacro:property name="wheel_mass" value="0.4" />
-  <xacro:property name="capota_car_length" value="0.2746" />      <!-- x axis  -->
-  <xacro:property name="capota_car_width" value="0.2124" />       <!-- y axis  -->
-  <xacro:property name="capota_car_height" value="0.0508" />      <!-- z axis  -->
-  <xacro:property name="capota_car_mass" value="0.25" />
+  <xacro:property name="capota_car_length" value="0.2746" />      <xacro:property name="capota_car_width" value="0.2124" />       <xacro:property name="capota_car_height" value="0.0508" />      <xacro:property name="capota_car_mass" value="0.25" />
   <xacro:property name="steering_cylinder_radius" value="0.01" />
   <xacro:property name="steering_cylinder_length" value="0.2124" />
   <xacro:property name="steering_cylinder_mass" value="0.05" />
-<!-- control parameters -->
-  <xacro:property name="back_wheels_velocity_limit" value="100.0" />
+<xacro:property name="back_wheels_velocity_limit" value="100.0" />
   <xacro:property name="steering_velocity_limit" value="100.0" />
-  <!-- Gazebo friction parameters -->
   <gazebo reference="base_link">
     <mu1>0.2</mu1>
@@ -40,4 +35,34 @@
     <mu2>100.0</mu2>
   </gazebo>
+  <gazebo reference="base_link">
+    <material>Gazebo/Green</material>
+  </gazebo>
+  <gazebo reference="capota">
+    <material>Gazebo/Green</material>
+  </gazebo>
+  <gazebo reference="steering_cylinder_link">
+    <material>Gazebo/DarkGrey</material>
+  </gazebo>
+  <gazebo reference="front_left_wheel_link">
+    <material>Gazebo/Yellow</material>
+  </gazebo>
+  <gazebo reference="front_right_wheel_link">
+    <material>Gazebo/Yellow</material>
+  </gazebo>
+  <gazebo reference="back_left_wheel_link">
+    <material>Gazebo/Yellow</material>
+  </gazebo>
+  <gazebo reference="back_right_wheel_link">
+    <material>Gazebo/Yellow</material>
+  </gazebo>
+  <gazebo reference="camera_link">
+    <material>Gazebo/Red</material>
+  </gazebo>
+ <material name="car_body_color"> <color rgba="0.8 0.1 0.1 1" /> </material>
+  <material name="car_capota_color"> <color rgba="0.1 0.1 0.8 1" /> </material>
+  <material name="steering_color"> <color rgba="0.3 0.3 0.3 1" /> </material>
+  <material name="wheel_main_color"> <color rgba="0.2 0.2 0.2 1" /> </material>
+  <material name="wheel_stripe_color"> <color rgba="1.0 1.0 0.0 1" /> </material>
+  <material name="camera_color"> <color rgba="0.1 0.1 0.1 1" /> </material>
   <material name="green">
     <color rgba="0 1 0 1" />
@@ -58,12 +83,5 @@
     </plugin>
   </gazebo>
-<!-- For bringing colors to the main simulation -->
- <gazebo>
-    <plugin name="gazebo_ros_material_plugin" filename="libgazebo_ros_api_plugin.so">
-      <robotNamespace>/car</robotNamespace>
-    </plugin>
-  </gazebo>
-  <!-- Dummy and Base Link -->
-  <link name="dummy"> </link>
+<link name="dummy"> </link>
   <joint name="dummy_joint" type="fixed">
     <parent link="dummy" />
@@ -75,5 +93,5 @@
         <box size="${car_length} ${car_width} ${car_height}" />
       </geometry>
-      <material name="green" />
+      <material name="car_body_color" />
     </visual>
     <collision>
@@ -93,11 +111,10 @@
     </inertial>
   </link>
-<!-- Capota of car -->
-  <link name="capota">
+<link name="capota">
     <visual>
       <geometry>
         <box size="${capota_car_length} ${capota_car_width} ${capota_car_height}" />
       </geometry>
-      <material name="light_green" />
+      <material name="car_capota_color" />
     </visual>
     <collision>
@@ -123,5 +140,4 @@
       rpy="0 0 0" />
   </joint>
-<!-- Steering cylinder axis -->
 <link name="steering_cylinder_link">
     <visual>
@@ -129,5 +145,5 @@
         <cylinder radius="${steering_cylinder_radius}" length="${steering_cylinder_length}"/>
       </geometry>
-      <material name="grey"/>
+      <material name="steering_color"/>
     </visual>
     <collision>
@@ -153,6 +169,4 @@
     <limit lower="${-pi/8}" upper="${pi/8}" effort="10.0" velocity="${steering_velocity_limit}"/>
   </joint>
-  <!-- Wheels -->
-  <!-- Front Left Wheel -->
   <link name="front_left_wheel_link">
     <visual>
@@ -183,6 +197,5 @@
     <axis xyz="0 0 1"/>
   </joint>
-<!-- Front Right Wheel -->
-  <link name="front_right_wheel_link">
+<link name="front_right_wheel_link">
     <visual>
       <geometry>
@@ -212,5 +225,4 @@
     <axis xyz="0 0 1"/>
   </joint>
-  <!-- back_left_wheel -->
   <link name="back_left_wheel_link">
     <visual>
@@ -243,5 +255,4 @@
     <limit effort="10.0" velocity="${back_wheels_velocity_limit}" />
   </joint>
-  <!-- back_right_wheel -->
   <link name="back_right_wheel_link">
     <visual>
@@ -275,10 +286,9 @@
     <limit effort="10.0" velocity="${back_wheels_velocity_limit}" />
   </joint>
-<!-- Camera -->
 <link name="camera_link">
     <visual>
       <geometry>
         <box size="0.02 0.02 0.02"/> </geometry>
-      <material name="grey"/>
+      <material name="camera_color"/>
     </visual>
     <collision>

Commit message: second checkpoint - lacking ramp

File: src/steering_car/urdf/car.xacro (robot description, xacro)
@@ -5,8 +5,8 @@
   <xacro:property name="car_width" value="0.2124" />
   <xacro:property name="car_height" value="0.0762" />
-  <xacro:property name="car_mass" value="2.0" />
+  <xacro:property name="car_mass" value="2.4" />
   <xacro:property name="wheel_radius" value="0.0508" />
   <xacro:property name="wheel_length" value="0.0508" />
-  <xacro:property name="wheel_mass" value="0.4" />
+  <xacro:property name="wheel_mass" value="0.6"/>
   <xacro:property name="capota_car_length" value="0.2746" />      <xacro:property name="capota_car_width" value="0.2124" />       <xacro:property name="capota_car_height" value="0.0508" />      <xacro:property name="capota_car_mass" value="0.25" />
   <xacro:property name="steering_cylinder_radius" value="0.01" />
@@ -167,5 +167,5 @@
     <origin xyz="${car_length/2-car_length/16} 0  ${-car_height/2}" rpy="${pi/2} 0 0"/>
     <axis xyz="0 1 0"/>
-    <limit lower="${-pi/8}" upper="${pi/8}" effort="10.0" velocity="${steering_velocity_limit}"/>
+    <limit lower="${-pi/16}" upper="${pi/16}" effort="10.0" velocity="${steering_velocity_limit}"/>
   </joint>
   <link name="front_left_wheel_link">

Commit message: Final documentation structure

File: src/steering_car/urdf/car.xacro (robot description, xacro)
@@ -9,5 +9,8 @@
   <xacro:property name="wheel_length" value="0.0508" />
   <xacro:property name="wheel_mass" value="0.6"/>
-  <xacro:property name="capota_car_length" value="0.2746" />      <xacro:property name="capota_car_width" value="0.2124" />       <xacro:property name="capota_car_height" value="0.0508" />      <xacro:property name="capota_car_mass" value="0.25" />
+  <xacro:property name="capota_car_length" value="0.2746" />
+  <xacro:property name="capota_car_width" value="0.2124" />
+  <xacro:property name="capota_car_height" value="0.0508" />
+  <xacro:property name="capota_car_mass" value="0.25" />
   <xacro:property name="steering_cylinder_radius" value="0.01" />
   <xacro:property name="steering_cylinder_length" value="0.2124" />
